File: kicad/air-quality-monitor.kicad_sch (KiCad schematic)
At the start: 30 parts, among them J1 USB-C power only, J2 SCD40 breakout, J3 OLED SSD1306, J4 SPS30, J5 Qwiic, J6 Qwiic, U1 AP2112K-3.3, U2 AP2112K-3.3, U3 ESP32-C6-DevKitC-1

Commit message: Rename the dev board header nets to DEVPIN_*
DEV_3V3 and 3V3_DEV were one character shuffle apart but sit on opposite sides of JP4, which makes the two easy to mix up.
Connections:
- net DEV_3V3 renamed DEVPIN_3V3
- net DEV_5V renamed DEVPIN_5V
- net DEV_GND1 renamed DEVPIN_GND1
- net DEV_GND2 renamed DEVPIN_GND2
- net DEV_IO21 renamed DEVPIN_IO21
- net DEV_IO22 renamed DEVPIN_IO22
Changed lines of the file:
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@@
 		)
 	)
-	(label "DEV_3V3"
+	(label "DEVPIN_3V3"
 		(at 190.5 171.45 90)
 		(effects
@@
 		)
 	)
-	(label "DEV_IO22"
+	(label "DEVPIN_IO22"
 		(at 220.98 125.73 0)
 		(effects
@@
 		)
 	)
-	(label "DEV_5V"
+	(label "DEVPIN_5V"
 		(at 246.38 124.46 180)
 		(effects
@@
 		)
 	)
-	(label "DEV_GND1"
+	(label "DEVPIN_GND1"
 		(at 180.34 148.59 180)
 		(effects
@@
 		)
 	)
-	(label "DEV_IO21"
+	(label "DEVPIN_IO21"
 		(at 246.38 154.94 180)
 		(effects
@@
 		)
 	)
-	(label "DEV_3V3"
+	(label "DEVPIN_3V3"
 		(at 177.8 171.45 90)
 		(effects
@@
 		)
 	)
-	(label "DEV_IO22"
+	(label "DEVPIN_IO22"
 		(at 246.38 165.1 180)
 		(effects
@@
 		)
 	)
-	(label "DEV_3V3"
+	(label "DEVPIN_3V3"
 		(at 246.38 114.3 180)
 		(effects
@@
 		)
 	)
-	(label "DEV_GND1"
+	(label "DEVPIN_GND1"
 		(at 246.38 134.62 180)
 		(effects
@@
 		)
 	)
-	(label "DEV_GND2"
+	(label "DEVPIN_GND2"
 		(at 246.38 144.78 180)
 		(effects
@@
 		)
 	)
-	(label "DEV_3V3"
+	(label "DEVPIN_3V3"
 		(at 180.34 113.03 180)
 		(effects
@@
 		)
 	)
-	(label "DEV_IO21"
+	(label "DEVPIN_IO21"
 		(at 220.98 128.27 0)
 		(effects
@@
 		)
 	)
-	(label "DEV_GND2"
+	(label "DEVPIN_GND2"
 		(at 220.98 113.03 0)
 		(effects
@@
 		)
 	)
-	(label "DEV_5V"
+	(label "DEVPIN_5V"
 		(at 180.34 146.05 180)
 		(effects
