File: kicad/air-quality-monitor.kicad_sch (KiCad schematic)
At the start: 30 parts, among them J1 USB-C power only, J2 SCD40 breakout, J3 OLED SSD1306, J4 SPS30, J5 Qwiic, J6 Qwiic, U1 AP2112K-3.3, U2 AP2112K-3.3, U3 ESP32-C6-DevKitC-1

Commit message: Show the power direction in the dev board net names
3V3_DEV comes out of the dev board and 5V_DEV goes into it, but the two names looked the same.

Co-Authored-By: Claude Opus 5.5 <noreply@anthropic.com>
Connections:
- net 3V3_DEV renamed 3V3_FROM_DEV
- net 5V_DEV renamed 5V_TO_DEV
Changed lines of the file:
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@@
 		)
 	)
-	(label "5V_DEV"
+	(label "5V_TO_DEV"
 		(at 261.62 124.46 0)
 		(effects
@@
 		)
 	)
-	(label "3V3_DEV"
+	(label "3V3_FROM_DEV"
 		(at 101.6 114.3 0)
 		(effects
@@
 		)
 	)
-	(label "3V3_DEV"
+	(label "3V3_FROM_DEV"
 		(at 261.62 114.3 0)
 		(effects
@@
 		)
 	)
-	(label "5V_DEV"
+	(label "5V_TO_DEV"
 		(at 165.1 66.04 0)
 		(effects
@@
 		)
 	)
-	(label "5V_DEV"
+	(label "5V_TO_DEV"
 		(at 163.83 53.34 0)
 		(effects
@@
 		)
 	)
-	(label "3V3_DEV"
+	(label "3V3_FROM_DEV"
 		(at 101.6 149.86 0)
 		(effects

Commit message: Say why the extra I2C pull-ups stay unfitted
The note only said the bus test decides, which hid that the SCD40 breakout already pulls the bus up. Moved up as well, because its second line ran into the 3V3_AUX labels.

Co-Authored-By: Claude Opus 5.5 <noreply@anthropic.com>
Other:
- note added: "Extra pull-ups, not fitted: the SCD40 breakout"
- note added: "already pulls SDA/SCL up (7.5k)."
- note removed: "Pull-ups: not fitted by default,"
- note removed: "decided by the bus test."
Changed lines of the file:
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@@
 		)
 	)
-	(text "Pull-ups: not fitted by default,"
+	(text "Extra pull-ups, not fitted: the SCD40 breakout"
 		(exclude_from_sim no)
-		(at 223.52 200.66 0)
+		(at 223.52 195.58 0)
 		(effects
 			(font
@@
 		)
 	)
-	(text "decided by the bus test."
+	(text "already pulls SDA/SCL up (7.5k)."
 		(exclude_from_sim no)
-		(at 223.52 204.47 0)
+		(at 223.52 199.39 0)
 		(effects
 			(font

Commit message: Say what R3 and R4 are for
Otherwise the optional footprints look pointless next to a note saying the breakout already has pull-ups.

Co-Authored-By: Claude Opus 5.5 <noreply@anthropic.com>
Other:
- note added: "R3/R4 are for a breakout without its own."
Changed lines of the file:
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@@
 	(text "Extra pull-ups, not fitted: the SCD40 breakout"
+		(exclude_from_sim no)
+		(at 223.52 191.77 0)
+		(effects
+			(font
+				(size 1.27 1.27)
+			)
+			(justify left bottom)
+		)
+	)
+	(text "already pulls SDA/SCL up (7.5k)."
 		(exclude_from_sim no)
 		(at 223.52 195.58 0)
@@
 		)
 	)
-	(text "already pulls SDA/SCL up (7.5k)."
+	(text "R3/R4 are for a breakout without its own."
 		(exclude_from_sim no)
 		(at 223.52 199.39 0)
